File: FitHome_atm90e32.sch (KiCad schematic (older format))
At the start: 39 parts, among them J1 PJ-002AH-SMT-TR, J2 Conn_01x09, U1 TRS35_3, U2 TRS35_3, U3 TPS62162DSGR, U4 ATM90E32, Y1 Crystal_GND2

Commit message: OSH Park - first build
Parts:
- C16, C4: value .033uF -> .033u
- J1: symbol FitHome_pwr_jack:PJ-002AH-SMT-TR -> FitHome_atm90e32-rescue:PJ-002AH-SMT-TR-FitHome_pwr_jack; PN CUI_PJ-002AH-SMT-TR -> PJ-002AH-SMT-TR
- J2: PN (none) -> X
- U1, U2: PN (none) -> SJ-3523-SMT-TR
- U4: symbol FitHome_atm90e32:ATM90E32 -> FitHome_atm90e32-rescue:ATM90E32-FitHome_atm90e32
Changed lines of the file:
@@
 $EndDescr
 $Comp
-L FitHome_atm90e32:ATM90E32 U4
+L FitHome_atm90e32-rescue:ATM90E32-FitHome_atm90e32 U4
 U 1 1 5CDDCE86
 P 8150 4150
@@
 F 2 "HappyDayEnergy:Audio-Jack" H 850 7400 50  0001 C CNN
 F 3 "" H 850 7400 50  0001 C CNN
+F 4 "SJ-3523-SMT-TR" H 850 7400 50  0001 C CNN "PN"
 	1    850  7400
 	1    0    0    -1
@@
 F 2 "HappyDayEnergy:Audio-Jack" H 2500 7400 50  0001 C CNN
 F 3 "" H 2500 7400 50  0001 C CNN
+F 4 "SJ-3523-SMT-TR" H 2500 7400 50  0001 C CNN "PN"
 	1    2500 7400
 	1    0    0    -1
@@
 Low Pass\nFilter
 $Comp
-L FitHome_pwr_jack:PJ-002AH-SMT-TR J1
+L FitHome_atm90e32-rescue:PJ-002AH-SMT-TR-FitHome_pwr_jack J1
 U 1 1 5CDEDA12
 P 1050 2500
@@
 F 2 "PJ-002AH-SMT-TR:CUI_PJ-002AH-SMT-TR" H 1050 2500 50  0001 L BNN
 F 3 "Manufacturer recommendations" H 1050 2500 50  0001 L BNN
-F 4 "CUI_PJ-002AH-SMT-TR" H 1050 2500 50  0001 C CNN "PN"
+F 4 "PJ-002AH-SMT-TR" H 1050 2500 50  0001 C CNN "PN"
 F 5 "CUI INC" H 1050 2500 50  0001 L BNN "Field4"
 	1    1050 2500
@@
 P 2750 3950
 F 0 "C4" H 2635 3904 50  0000 R CNN
-F 1 ".033uF" H 2635 3995 50  0000 R CNN
+F 1 ".033u" H 2635 3995 50  0000 R CNN
 F 2 "Capacitor_SMD:C_0805_2012Metric" H 2788 3800 50  0001 C CNN
 F 3 "" H 2750 3950 50  0001 C CNN
@@
 F 2 "HappyDayEnergy:9Pin-bb" H 10600 5400 50  0001 C CNN
 F 3 "~" H 10600 5400 50  0001 C CNN
+F 4 "X" H 10600 5400 50  0001 C CNN "PN"
 	1    10600 5400
 	1    0    0    -1
@@
 P 4200 3900
 F 0 "C16" H 4085 3854 50  0000 R CNN
-F 1 ".033uF" H 4085 3945 50  0000 R CNN
+F 1 ".033u" H 4085 3945 50  0000 R CNN
 F 2 "Capacitor_SMD:C_0805_2012Metric" H 4238 3750 50  0001 C CNN
 F 3 "" H 4200 3900 50  0001 C CNN
